File: pcb/wifi-modem.kicad_pcb (KiCad board)
At the start: 2 copper layers, 69 x 67 mm, 58 parts, among them J1 USB_B, J2 Conn_01x03, J3 RS232 DB9, Q1 Q_NPN_BEC, Q2 Q_NPN_BEC, SW1 SW_Push, U1 ESP-12F, U2 74HC245, U3 LM1117-3.3, U4 FT232RL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

Commit message: Finished layout for 2.1
Parts:
- added C11: 100n, Capacitor_SMD:C_0805_2012Metric_Pad1.15x1.40mm_HandSolder, F.Cu at (75.8, 114.0)
- moved C15 72.8 mm to (88.6, 80.2), turned to 270 degrees
- moved C17 70.6 mm to (73.4, 84.4), turned to 180 degrees
- moved C13 69.1 mm to (84.4, 79.2), turned to 270 degrees
- moved C14 66.0 mm to (86.6, 80.2), turned to 270 degrees
- moved C7 63.1 mm to (88.8, 93.0), turned to 270 degrees
- moved C6 59.4 mm to (80.8, 87.2), turned to 180 degrees
- moved C5 52.2 mm to (81.0, 99.0)
- moved C16 48.3 mm to (54.2, 109.0), turned to 270 degrees
- moved C10 42.4 mm to (75.8, 110.0), turned to 270 degrees
- moved C12 31.2 mm to (86.5, 119.5)
- moved C8 30.5 mm to (78.5, 119.5)
- moved C9 27.0 mm to (82.5, 119.5)
- moved JP1 3.49 mm to (93.1, 66.2), turned to 90 degrees
- moved FB1 2.44 mm to (87.6, 77.2)
Routing:
- net +3V3: track 11.8 -> 159.1 mm, vias 0 -> 5
- net ESP_GPIO0: track 16.9 -> 117.6 mm, vias 0 -> 3
- net ESP_UART0_RXD: track 0.00 -> 75.2 mm, vias 0 -> 3
- net ESP_RST_N: track 0.00 -> 75.0 mm, vias 0 -> 2
- net ESP_GPIO15_UART0_RTS: track 0.00 -> 74.4 mm, vias 0 -> 3
- net +5V: track 93.4 -> 148.3 mm
- net ESP_EN: track 0.00 -> 49.5 mm
- net GND: track 13.9 -> 62.1 mm, vias 5 -> 69
- net ESP_GPIO4: track 0.00 -> 36.7 mm, vias 0 -> 2
- net ESP_GPIO5: track 0.00 -> 36.1 mm, vias 0 -> 2
- net 3V3_TTL_HDR_RXD: track 0.00 -> 32.6 mm, vias 0 -> 1
- net MAX232_RXD: track 0.00 -> 21.7 mm
- net FT232_RTS: track 0.00 -> 19.8 mm
- net FT232_DTR: track 0.00 -> 17.5 mm
- net 3V3_TTL_TXD: track 109.9 -> 124.4 mm
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Other:
- board text added: "WiFi Modem Rev. 2.1"
- board text removed: "WiFi Modem Rev. 2.0"

Commit message: Final tweaks
Routing:
- net GND: track 62.1 -> 59.4 mm
- net ESP_GPIO14: track 48.0 -> 48.9 mm
- net MAX232_RXD: track 21.7 -> 22.3 mm
